File: EAGLE/sr42/sr42-revB-kbd.sch (EAGLE design)
At the start: 184 parts, among them M0 74HC589A_DT, M1 74HC589A_DT, M2 74HC589A_DT, M3 74HC589A_DT, M4 74HC589A_DT, M5 74HC589A_DT, U1 2N7002

Commit message: ·
Parts:
- U$1: value VR42_MLB_FOOTPRINT -> SR42_MLB_FOOTPRINT; device __temp_to_delete:VR42_MLB_FOOTPRINT -> __temp_to_delete:SR42_MLB_FOOTPRINT
Changed lines of the file:
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@@
 <part name="SUPPLY2" library="SparkFun-PowerSymbols" library_urn="urn:adsk.eagle:library:530" deviceset="VCC_1" device="" value="5V"/>
 <part name="SUPPLY3" library="SparkFun-PowerSymbols" library_urn="urn:adsk.eagle:library:530" deviceset="VCC_1" device="" value="5V"/>
-<part name="U$1" library="__temp_to_delete" deviceset="VR42_MLB_FOOTPRINT" device=""/>
+<part name="U$1" library="__temp_to_delete" deviceset="SR42_MLB_FOOTPRINT" device=""/>
 <part name="U1" library="__temp_to_delete" deviceset="2N7002" device=""/>
 <part name="U$2" library="__temp_to_delete" deviceset="UBD_FOOTPRINT" device=""/>
