File: EAGLE/sr42/sr42-revB-mlb.brd (EAGLE design)
At the start: 70 x 30 mm, 87 parts, among them SW2 KMR2, U1 2N7002, U2 2N7002, U3 74AHCT1G125GW, U33 USB3300-EZK, X1 12MHz, X2 32.768MHz, X3 24MHz

Commit message: ·
Parts:
- U$1: value VR42_MLB_FOOTPRINT -> SR42_MLB_FOOTPRINT; device __temp_to_delete:VR42_MLB_FOOTPRINT -> __temp_to_delete:SR42_MLB_FOOTPRINT
- moved LOGO1 8.60 mm to (61.8, 21.2)
Other:
- board text added: "(c) 2024 Silvino Rodrigues"
- board text added: "SR42 Keyboard MLB"
- board text added: "https://c1k.it/sr42"
- board text removed: "(c) 2024 Vino Rodrigues"
- board text removed: "VR42 Keyboard MLB"
- board text removed: "https://c1k.it/vr42"
Changed lines of the file:
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@@
 <drawing>
 <settings>
-<setting alwaysvectorfont="no"/>
+<setting alwaysvectorfont="yes"/>
 <setting verticaltext="up"/>
 </settings>
-<grid distance="1" unitdist="mm" unit="mm" style="dots" multiple="2" display="yes" altdistance="0.0025" altunitdist="mm" altunit="mm"/>
+<grid distance="1" unitdist="mm" unit="mm" style="dots" multiple="2" display="yes" altdistance="0.1" altunitdist="mm" altunit="mm"/>
 <layers>
 <layer number="1" name="Top" color="4" fill="1" visible="yes" active="yes"/>
@@
 <wire x1="70" y1="3" x2="67" y2="0" width="0" layer="20" curve="-90"/>
 <wire x1="70" y1="27" x2="67" y2="30" width="0" layer="20" curve="90"/>
-<text x="61.155" y="1.975" size="1.5" layer="22" rot="MR0">VR42 Keyboard MLB</text>
-<text x="68.675" y="22.225" size="1.27" layer="22" rot="MR0">(c) 2024 Vino Rodrigues</text>
+<text x="61.155" y="1.975" size="1.5" layer="22" rot="MR0">SR42 Keyboard MLB</text>
+<text x="29.675" y="3.225" size="1.27" layer="22" rot="MR0">(c) 2024 Silvino Rodrigues</text>
 <text x="3.95" y="8" size="0.8128" layer="25" align="bottom-center">VCC</text>
 <text x="4" y="7" size="0.8128" layer="25" align="bottom-center">RST</text>
@@
 <wire x1="5.15" y1="6.4" x2="6.6" y2="3.55" width="0.0762" layer="25"/>
 <text x="63.2" y="20.3" size="0.8128" layer="25" align="bottom-center">(c) 2024
-Vino Rodrigues</text>
+Silvino Rodrigues</text>
 <text x="8.3" y="9.45" size="0.8128" layer="26" rot="MR0" align="bottom-center">VCC</text>
 <text x="1.55" y="12" size="0.8128" layer="26" rot="MR0" align="bottom-center">RST</text>
@@
 <wire x1="62" y1="26.5" x2="62" y2="27" width="0.1524" layer="25"/>
 <wire x1="63" y1="3.5" x2="63" y2="4" width="0.1524" layer="25"/>
-<text x="68.7" y="18.5" size="1.27" layer="22" rot="MR0">https://c1k.it/vr42</text>
+<text x="68.7" y="17.5" size="1.27" layer="22" rot="MR0">https://c1k.it/sr42</text>
 <wire x1="63" y1="4" x2="63" y2="4.5" width="0.1524" layer="21"/>
 <wire x1="63" y1="4.5" x2="63.5" y2="4.5" width="0.1524" layer="21"/>
@@
 <attribute name="NAME" x="29.814465625" y="9.692890625" size="0.8128" layer="25" ratio="6" rot="SR45"/>
 </element>
-<element name="U$1" library="__temp_to_delete" package="VR42_MLB_FOOTPRINT" value="VR42_MLB_FOOTPRINT" x="35" y="15" smashed="yes"/>
+<element name="U$1" library="__temp_to_delete" package="SR42_MLB_FOOTPRINT" value="SR42_MLB_FOOTPRINT" x="35" y="15" smashed="yes"/>
 <element name="UDB" library="ts_keyboards" package="MOLEX_781710004" value="" x="67" y="15" smashed="yes" rot="R90">
 <attribute name="NAME" x="63.456" y="12.702" size="0.8128" layer="25" font="vector" rot="R270"/>
@@
 <element name="U$5" library="ts_keyboards" package="MOUNTING-HOLE" value="MOUNTING-HOLE" x="67" y="3" smashed="yes"/>
 <element name="U$6" library="random_logos" package="TECSMITH-NAME" value="TECSMITH-LOGOLONG" x="62.83" y="7.7" smashed="yes" rot="MR0"/>
-<element name="LOGO1" library="random_logos" package="OSHW-LOGO-M" value="OSHW-LOGOM" x="54.75" y="26.25" smashed="yes" rot="MR0"/>
+<element name="LOGO1" library="random_logos" package="OSHW-LOGO-M" value="OSHW-LOGOM" x="61.75" y="21.25" smashed="yes" rot="MR0"/>
 <element name="TC" library="__untitled" package="TC2030-MCP-NL" value="" x="7.55" y="7" smashed="yes" rot="R270">
 <attribute name="NAME" x="7.5" y="2.5" size="1.016" layer="25" rot="R180" align="bottom-center"/>
