File: EAGLE/sr42/sr42-revB-mlb.sch (EAGLE design)
At the start: 87 parts, among them SW2 KMR2, U1 2N7002, U2 2N7002, U3 74AHCT1G125GW, U33 USB3300-EZK, X1 12MHz, X2 32.768MHz, X3 24MHz

Commit message: ·
Parts:
- U$1: value VR42_MLB_FOOTPRINT -> SR42_MLB_FOOTPRINT; device __temp_to_delete:VR42_MLB_FOOTPRINT -> __temp_to_delete:SR42_MLB_FOOTPRINT
Changed lines of the file:
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@@
 <part name="SUPPLY9" library="SparkFun-PowerSymbols" library_urn="urn:adsk.eagle:library:530" deviceset="VCC_2" device="" value="3V3"/>
 <part name="SUPPLY10" library="supply2" library_urn="urn:adsk.eagle:library:372" deviceset="GND" device=""/>
-<part name="U$1" library="__temp_to_delete" deviceset="VR42_MLB_FOOTPRINT" device=""/>
+<part name="U$1" library="__temp_to_delete" deviceset="SR42_MLB_FOOTPRINT" device=""/>
 <part name="UDB" library="ts_keyboards" deviceset="UBD-S1_C4" device=""/>
 <part name="C18" library="rcl" library_urn="urn:adsk.eagle:library:334" deviceset="C-EU" device="C0603" package3d_urn="urn:adsk.eagle:package:23616/2" value="1uF"/>
