File: KiCAD/udk_module_stm32f405/udk_module_stm32f405.kicad_pcb (KiCad board)
At the start: 4 copper layers, 54 x 38 mm, 79 parts, among them J1 5V, J2 USB_C_Receptacle, J3 QWIIC, J4 SPI, J5 TC2030_SWD, J6 CONN, J7 ARGB, U1 AMS1117-3.3, U2 STM32F405RGTx, U3 NC7SZ125M5X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

Commit message: UDK Version
Parts:
- moved D2 0.95 mm to (116.8, 49.0)
- moved BOOT1 0.75 mm to (120.5, 51.5)
Routing:
- net GNDREF: track 47.1 -> 40.3 mm
- net +3V3: track 244.3 -> 242.2 mm
- net Net-(BOOT1-B): track 2.41 -> 3.39 mm
- net SWCLK: track 11.0 -> 10.0 mm
- net SWDIO: track 17.5 -> 16.6 mm
- net GND: track 106.9 -> 106.3 mm, vias 54 -> 55

Commit message: move rgb to spi pin
Connections:
- J6 pad 4: CON4 -> TX/CON4
- J6 pad 5: CON5 -> RX/CON5
- U2 pad 42: unconnected-(U2-PA9-Pad42) -> TX/CON4
- U2 pad 43: unconnected-(U2-PA10-Pad43) -> RX/CON5
- U2 pad 51: CON5 -> Do_not_use_1
- U2 pad 52: CON4 -> unconnected-(U2-PC11-Pad52)
- U2 pad 53: RGB-EN1 -> RGB
- U2 pad 54: unconnected-(U2-PD2-Pad54) -> RGB-EN1
- U2 pad 59: RGB -> unconnected-(U2-PB7-Pad59)
Routing:
- net CON5: track 15.9 -> 0.00 mm, vias 2 -> 0
- net CON4: track 15.9 -> 0.00 mm, vias 2 -> 0
- net TX/CON4: track 0.00 -> 12.9 mm, vias 0 -> 2
- net RX/CON5: track 0.00 -> 12.9 mm, vias 0 -> 2
- net SS/MATRIX-CS: track 26.4 -> 33.7 mm
- net RGB: track 7.09 -> 4.59 mm
- net +3V3: track 242.2 -> 242.8 mm
- net GND: track 106.3 -> 106.9 mm, vias 55 -> 56
