File: KiCAD/udk_module_stm32f405/udk_module_stm32f405.kicad_sch (KiCad schematic)
At the start: 33 parts, among them J1 USB_C_Receptacle, J2 5V, J3 ARGB, J4 QWIIC, J5 CONN, J6 SPI, U1 AMS1117-3.3, U2 NC7SZ125M5X, U3 STM32F405RGTx, U4 USB3300-EZK, U5 TS3USB30EDGSR

Commit message: wip-2025-11-27
Parts:
- removed U3: STM32F405RGTx, Package_QFP:LQFP-64_10x10mm_P0.5mm, symbol MCU_ST_STM32F4:STM32F405RGTx
- removed U4: USB3300-EZK, Package_DFN_QFN:QFN-32-1EP_5x5mm_P0.5mm_EP3.45x3.45mm, symbol Interface_USB:USB3300-EZK
- added BOOT1: SW-BOOT, Button_Switch_SMD:SW_SPDT_Shouhan_MSK12C02, symbol ts-keyboard-lib:SW_SPDT
- added C10, C8: 20p, Capacitor_SMD:C_0603_1608Metric, symbol Device:C_Small
- added C11, C12, C7, C9: 100n, Capacitor_SMD:C_0603_1608Metric, symbol Device:C_Small
- added C13: 10n, Capacitor_SMD:C_0603_1608Metric, symbol Device:C_Small
- added C14, C16: 12p, Capacitor_SMD:C_0603_1608Metric, symbol Device:C_Small
- added C15: 1u, Capacitor_SMD:C_0603_1608Metric, symbol Device:C_Small
- added C18, C21: 2u2, Capacitor_SMD:C_0603_1608Metric, symbol PCM_SparkFun-Capacitor:C
- added C19, C20, C22, C24, C25, C27, C32: 100n, Capacitor_SMD:C_0603_1608Metric, symbol PCM_SparkFun-Capacitor:C
- added C23: 1u, Capacitor_SMD:C_0603_1608Metric, symbol PCM_SparkFun-Capacitor:C
- added C26, C28: 9p, Capacitor_SMD:C_0603_1608Metric, symbol PCM_SparkFun-Capacitor:C
- added C29, C30, C31: 4u7, Capacitor_SMD:C_0603_1608Metric, symbol PCM_SparkFun-Capacitor:C
- added D2: Blue, PCM_SparkFun-LED:LED_0603_1608Metric_Blue, symbol PCM_SparkFun-LED:LED_Blue_0603
- added FB2: 1kΩ@100MHz, Inductor_SMD:L_0603_1608Metric, symbol Device:FerriteBead_Small
- added J5: TC2030_SWD, PCM_marbastlib-various:CON_TC2030_outlined, symbol PCM_marbastlib-various:TC2030_SWD
- added R10: 12K, Resistor_SMD:R_0603_1608Metric, symbol Device:R
- added R4, R6, R8: 10K, Resistor_SMD:R_0603_1608Metric, symbol Device:R
- added R9: 820R, Resistor_SMD:R_0603_1608Metric, symbol Device:R
- added U2: STM32F405RGTx, Package_QFP:LQFP-64_10x10mm_P0.5mm, symbol ts-kb-mcus-lib:STM32F405RGTx
- added U4: MB85RS64, Package_SO:SOIC-8_5.3x5.3mm_P1.27mm, symbol Memory_NVRAM:MB85RS64
- added U6: USB3300-EZK, Package_DFN_QFN:QFN-32-1EP_5x5mm_P0.5mm_EP3.45x3.45mm, symbol ts-kb-mcus-lib:USB3300-EZK
- added Y1: 25MHz 20pF SMD3225-4P, Crystal:Crystal_SMD_3225-4Pin_3.2x2.5mm, symbol Device:Crystal_GND24_Small
- added Y2: 32.768kHz 12.5pF SMD3215-2P, Crystal:Crystal_SMD_3215-2Pin_3.2x1.5mm, symbol Device:Crystal_Small
- added Y3: 24MHz, Crystal:Crystal_SMD_3225-4Pin_3.2x2.5mm, symbol Device:Crystal_GND24_Small
- added ~{RST}1: SW-RESET, Button_Switch_SMD:SW_SPST_CK_KMS2xxGP, symbol atelier-microcontrollers:SW_Push_Small
- C1: renamed from C4; footprint PCM_SparkFun-Capacitor:C_0603_1608Metric -> Capacitor_SMD:C_0603_1608Metric; PROD_ID CAP-00867 -> (none); Tolerance 10% -> (none); Voltage 50V -> (none)
- C17: renamed from C7; footprint PCM_SparkFun-Capacitor:C_0603_1608Metric -> Capacitor_SMD:C_0603_1608Metric; PROD_ID CAP-00000 -> (none); Tolerance 100% -> (none); Voltage 1kV -> (none)
- C2: footprint PCM_SparkFun-Capacitor:C_0603_1608Metric -> Capacitor_SMD:C_0603_1608Metric; PROD_ID CAP-13930 -> (none); Tolerance 10% -> (none); Voltage 16V -> (none)
- C4: renamed from C5; footprint PCM_SparkFun-Capacitor:C_0603_1608Metric -> Capacitor_SMD:C_0603_1608Metric; PROD_ID CAP-00867 -> (none); Tolerance 10% -> (none); Voltage 50V -> (none)
- C5: renamed from C6; footprint PCM_SparkFun-Capacitor:C_0603_1608Metric -> Capacitor_SMD:C_0603_1608Metric; PROD_ID CAP-14106 -> (none); Tolerance 20% -> (none); Voltage 35V -> (none)
- C6: renamed from C3; footprint PCM_SparkFun-Capacitor:C_0603_1608Metric -> Capacitor_SMD:C_0603_1608Metric; PROD_ID CAP-13930 -> (none); Tolerance 10% -> (none); Voltage 16V -> (none)
- renumbered C1 to C3, J2 to J1, J1 to J2, J4 to J3, J6 to J4, J5 to J6, J3 to J7, R3 to R1, R1 to R2, R2 to R3, R4 to R5, R5 to R7, U2 to U3
Connections:
- net +3.3V is gone; now on net +3V3: C6.1, D1.2 (A), J3.2, J4.2, U1.2 (VO)
- net +5V: now also C23.1, R9.2
- net CON4: now also U2.42 (PA9)
- net CON5: now also U2.43 (PA10)
- net D+: now also U5.4 (D+)
- net D-: now also U5.6 (D-)
- net GND: now also U5.5 (GND), U5.9 (~{OE}), BOOT1.3 (C), C10.1, C11.1, C12.1, C13.1, C14.1, C15.1, C16.1, C18.2, C19.2, C20.2, C21.2, C22.2, C23.2, C24.2, C25.2, C26.2, C27.2, C28.2, C29.2, C30.2, C31.2, C32.2, C7.1, C8.1, C9.1, D2.1 (K), J5.5 (GND), R10.2, U2.12 (VSSA), U2.18 (VSS), U2.63 (VSS), U4.3 (~{WP}), U4.4 (GND), U4.7 (~{HOLD}), U6.1 (GND), U6.2 (GND), U6.33 (GND), Y1.2, Y1.4, Y3.2, Y3.4, ~{RST}1.2
- net RGB: now also R5.1, U2.59 (PB7)
- net SCK: now also U2.55 (PB3), U4.6 (SCK)
- net USB_SELECT: now reaches U5.1 (S)
- net USB_SELECT: now also U2.62 (PB9)
- net +3V3: now reaches U5.10 (VCC)
- net +3V3: now also BOOT1.1 (A), C11.2, C12.2, C20.1, C22.1, C24.1, C25.1, C27.1, C32.1, C7.2, C9.2, FB2.1, J5.1 (VCC), R6.1, U2.1 (VBAT), U2.19 (VDD), U2.32 (VDD), U2.48 (VDD), U2.64 (VDD), U4.8 (VDD), U6.16 (VDD3.3), U6.25 (VDD3.3), U6.30 (VDD3.3), U6.31 (REG_EN), U6.6 (VDD3.3)
- net USB-D1+: now reaches U5.2 (D1+)
- net USB-D1+: now also U2.45 (PA12)
- net USB-D2+: now reaches U5.3 (D2+)
- net USB-D2+: now also U6.7 (DP)
- net USB-D2-: now reaches U5.7 (D2-)
- net USB-D2-: now also U6.8 (DM)
- net USB-D1-: now reaches U5.8 (D1-)
- net USB-D1-: now also U2.44 (PA11)
- net CON1 renamed ADC1/WKUP/CON1
- net ADC1/WKUP/CON1: now also U2.14 (PA0)
- net CON2 renamed ADC2/CON2
- net ADC2/CON2: now also U2.15 (PA1)
- net CON3 renamed RGB-EN/ADC3
- net RGB-EN/ADC3: now also U2.16 (PA2)
- net PICO renamed MISO
- net MISO: now also U2.22 (PA6), U4.2 (SO)
- net POCI renamed MOSI
- net MOSI: now also U2.23 (PA7), U4.5 (SI)
- net SS renamed SS/MATRIX-CS
- net SS/MATRIX-CS: now also U2.50 (PA15)
- new net: BOOT1.2 (B), R8.2
- new net: C18.1, U2.31 (VCAP_1)
- new net: R10.1, U6.32 (RBIAS)
- new net: R9.1, U6.4 (VBUS)
- new net: D2.2 (A), R4.2
- new net: C21.1, U2.47 (VCAP_2)
- new net +1V8: C30.1, C31.1, U6.15 (VDD1.8), U6.26 (VDD1.8)
- new net BOOT0: R8.1, U2.60 (BOOT0)
- new net CLK: U2.21 (PA5), U6.14 (CLKOUT)
- new net DATA0: U2.17 (PA3), U6.24 (DATA0)
- new net DATA1: U2.26 (PB0), U6.23 (DATA1)
- new net DATA2: U2.27 (PB1), U6.22 (DATA2)
- new net DATA3: U2.29 (PB10), U6.21 (DATA3)
- new net DATA4: U2.30 (PB11), U6.20 (DATA4)
- new net DATA5: U2.33 (PB12), U6.19 (DATA5)
- new net DATA6: U2.34 (PB13), U6.18 (DATA6)
- new net DATA7: U2.57 (PB5), U6.17 (DATA7)
- new net DIR: U2.10 (PC2), U6.12 (DIR)
- new net EEPROM-CS: U2.39 (PC8), U4.1 (~{CS})
- new net NXT: U2.11 (PC3), U6.11 (NXT)
- new net OSC-IN: C8.2, U2.5 (PH0), Y1.1
- new net OSC-OUT: C10.2, U2.6 (PH1), Y1.3
- new net OSC32-IN: C14.2, U2.3 (PC14), Y2.1
- new net OSC32-OUT: C16.2, U2.4 (PC15), Y2.2
- new net STATUS-LED: R4.1, U2.40 (PC9)
- new net STP: U2.8 (PC0), U6.13 (STP)
- new net SWCLK: J5.4 (SWCLK), U2.49 (PA14)
- new net SWDIO: J5.2 (SWDIO), U2.46 (PA13)
- new net VDDA: C13.2, C15.2, FB2.2, U2.13 (VDDA)
- new net VDDA1.8: C29.1, U6.29 (VDDA1.8)
- new net XI: C28.1, U6.28 (XI), Y3.1
- new net XO: C26.1, U6.27 (XO), Y3.3
- new net ~{RST}: C19.1, J5.3 (~{RST}), R6.2, U2.7 (NRST), ~{RST}1.1
- no-connect marks 0 -> 25
Other:
- note added: "HIGH-SPEED USB"
- moved on the sheet: C17, C2, C6, J1, J3, J4, J6, J7, PTC1, R5, R7, U3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

Commit message: wip-2025-11-28
Parts:
- added C45: 100n, Capacitor_SMD:C_0603_1608Metric, symbol ts-kicad-lib:C
- added R49: 100R, Resistor_SMD:R_0603_1608Metric, symbol ts-kicad-lib:R
- added RLY1: TPS22810, Package_TO_SOT_SMD:SOT-23-6, symbol ts-kicad-lib:TPS22810
- added U7: SN74LVC1G14DBV, Package_TO_SOT_SMD:SOT-23-5, symbol ts-kicad-lib:SN74LVC1G14DBV
Connections:
- net +3V3: now also U7.5
- net +5V: now also C45.2, RLY1.1 (VIN); no longer C17.1, J7.3, U3.5 (VCC)
- net CON4: now also U2.52 (PC11); no longer U2.42 (PA9)
- net CON5: now also U2.51 (PC10); no longer U2.43 (PA10)
- net GND: now also C45.1, RLY1.2 (GND), U7.3; no longer U3.1 (~{OE})
- net SCL: now also U2.41 (PA8)
- net SDA: now also U2.40 (PC9)
- net STATUS-LED: now also U2.20 (PA4); no longer U2.40 (PC9)
- net RGB-EN1: now reaches U2.53 (PC12)
- net RGB-EN1: now also RLY1.3 (EN/VLO), U7.2
- net +1V8: no longer names the net of C30.1, U6.15 (VDD1.8)
- net +1V8: no longer C31.1, U6.26 (VDD1.8)
- net RGB-EN/ADC3 renamed RGB-EN2/ADC3
- net VDDA1.8: no longer names the net of C29.1, U6.29 (VDDA1.8)
- new net: R49.2, RLY1.5 (QOD)
- new net: C31.1, U6.26 (VDD1.8)
- new net VLED: C17.1, J7.3, R49.1, RLY1.6 (VOUT), U3.5 (VCC)
- new net ~{RGB-EN1}: U3.1 (~{OE}), U7.4
- no-connect marks 25 -> 23
Other:
- moved on the sheet: BOOT1, C29, C30, C31, C32, H1, H2, H3, H4, H5, H6, R8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

Commit message: UDK Version
Other:
- moved on the sheet: C18
Changed lines of the file:
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@@
 	(wire
 		(pts
-			(xy 142.24 33.02) (xy 142.24 35.56)
+			(xy 142.24 30.48) (xy 142.24 35.56)
 		)
 		(stroke
@@
 	(wire
 		(pts
-			(xy 172.72 83.82) (xy 175.26 83.82)
+			(xy 172.72 83.82) (xy 177.8 83.82)
 		)
 		(stroke
@@
 	(wire
 		(pts
-			(xy 157.48 93.98) (xy 157.48 96.52)
+			(xy 157.48 93.98) (xy 157.48 99.06)
 		)
 		(stroke
@@
 	(wire
 		(pts
+			(xy 124.46 93.98) (xy 124.46 99.06)
+		)
+		(stroke
+			(width 0)
+			(type default)
+		)
+	)
+	(wire
+		(pts
 			(xy 246.38 106.68) (xy 246.38 99.06)
 		)
@@
 	(wire
 		(pts
-			(xy 147.32 93.98) (xy 147.32 96.52)
+			(xy 147.32 93.98) (xy 147.32 99.06)
 		)
 		(stroke
@@
 	(wire
 		(pts
-			(xy 154.94 93.98) (xy 154.94 96.52)
+			(xy 154.94 93.98) (xy 154.94 99.06)
 		)
 		(stroke
@@
 	(wire
 		(pts
-			(xy 172.72 81.28) (xy 175.26 81.28)
-		)
-		(stroke
-			(width 0)
-			(type default)
-		)
-	)
-	(wire
-		(pts
 			(xy 266.7 48.26) (xy 269.24 48.26)
 		)
@@
 	(wire
 		(pts
-			(xy 160.02 93.98) (xy 160.02 104.14)
+			(xy 160.02 93.98) (xy 160.02 106.68)
 		)
 		(stroke
@@
 	(wire
 		(pts
-			(xy 124.46 93.98) (xy 124.46 96.52)
-		)
-		(stroke
-			(width 0)
-			(type default)
-		)
-	)
-	(wire
-		(pts
 			(xy 22.86 154.94) (xy 38.1 154.94)
 		)
@@
 	(wire
 		(pts
-			(xy 149.86 93.98) (xy 149.86 96.52)
+			(xy 149.86 93.98) (xy 149.86 99.06)
 		)
 		(stroke
@@
 	(wire
 		(pts
+			(xy 172.72 81.28) (xy 177.8 81.28)
+		)
+		(stroke
+			(width 0)
+			(type default)
+		)
+	)
+	(wire
+		(pts
 			(xy 60.96 180.34) (xy 60.96 182.88)
 		)
@@
 		)
 	)
+	(label "D0"
+		(at 124.46 97.79 90)
+		(effects
+			(font
+				(size 1.27 1.27)
+			)
+			(justify left bottom)
+		)
+	)
 	(label "D-"
 		(at 35.56 27.94 0)
@@
 		)
 	)
+	(label "D3"
+		(at 154.94 97.79 90)
+		(effects
+			(font
+				(size 1.27 1.27)
+			)
+			(justify left bottom)
+		)
+	)
 	(label "D+"
 		(at 35.56 30.48 0)
@@
 		)
 	)
+	(label "D6"
+		(at 173.99 81.28 0)
+		(effects
+			(font
+				(size 1.27 1.27)
+			)
+			(justify left bottom)
+		)
+	)
 	(label "CC2"
 		(at 35.56 35.56 0)
@@
 		)
 	)
+	(label "D5"
+		(at 173.99 83.82 0)
+		(effects
+			(font
+				(size 1.27 1.27)
+			)
+			(justify left bottom)
+		)
+	)
+	(label "D7"
+		(at 142.24 34.29 90)
+		(effects
+			(font
+				(size 1.27 1.27)
+			)
+			(justify left bottom)
+		)
+	)
 	(label "CC1"
 		(at 35.56 33.02 0)
@@
 		)
 	)
+	(label "D1"
+		(at 147.32 97.79 90)
+		(effects
+			(font
+				(size 1.27 1.27)
+			)
+			(justify left bottom)
+		)
+	)
+	(label "D2"
+		(at 149.86 97.79 90)
+		(effects
+			(font
+				(size 1.27 1.27)
+			)
+			(justify left bottom)
+		)
+	)
 	(label "15"
 		(at 266.7 76.2 0)
@@
 		)
 	)
+	(label "D4"
+		(at 157.48 97.79 90)
+		(effects
+			(font
+				(size 1.27 1.27)
+			)
+			(justify left bottom)
+		)
+	)
 	(global_label "RGB"
 		(shape input)
@@
 	(global_label "DATA7"
 		(shape input)
-		(at 142.24 33.02 90)
+		(at 142.24 30.48 90)
 		(fields_autoplaced yes)
 		(effects
@@
 		)
 		(property "Intersheetrefs" "${INTERSHEET_REFS}"
-			(at 142.24 24.4105 90)
+			(at 142.24 21.8705 90)
 			(effects
 				(font
@@
 	(global_label "DATA2"
 		(shape input)
-		(at 149.86 96.52 270)
+		(at 149.86 99.06 270)
 		(fields_autoplaced yes)
 		(effects
@@
 		)
 		(property "Intersheetrefs" "${INTERSHEET_REFS}"
-			(at 149.86 105.1295 90)
+			(at 149.86 107.6695 90)
 			(effects
 				(font
@@
 	(global_label "DATA6"
 		(shape input)
-		(at 175.26 81.28 0)
+		(at 177.8 81.28 0)
 		(fields_autoplaced yes)
 		(effects
@@
 		)
 		(property "Intersheetrefs" "${INTERSHEET_REFS}"
-			(at 183.8695 81.28 0)
+			(at 186.4095 81.28 0)
 			(effects
 				(font
@@
 	(global_label "DATA3"
 		(shape input)
-		(at 154.94 96.52 270)
+		(at 154.94 99.06 270)
 		(fields_autoplaced yes)
 		(effects
@@
 		)
 		(property "Intersheetrefs" "${INTERSHEET_REFS}"
-			(at 154.94 105.1295 90)
+			(at 154.94 107.6695 90)
 			(effects
 				(font
@@
 	(global_label "DATA1"
 		(shape input)
-		(at 147.32 96.52 270)
+		(at 147.32 99.06 270)
 		(fields_autoplaced yes)
 		(effects
@@
 		)
 		(property "Intersheetrefs" "${INTERSHEET_REFS}"
-			(at 147.32 105.1295 90)
+			(at 147.32 107.6695 90)
 			(effects
 				(font
@@
 	(global_label "DATA4"
 		(shape input)
-		(at 157.48 96.52 270)
+		(at 157.48 99.06 270)
 		(fields_autoplaced yes)
 		(effects
@@
 		)
 		(property "Intersheetrefs" "${INTERSHEET_REFS}"
-			(at 157.48 105.1295 90)
+			(at 157.48 107.6695 90)
 			(effects
 				(font
@@
 	(global_label "DATA5"
 		(shape input)
-		(at 175.26 83.82 0)
+		(at 177.8 83.82 0)
 		(fields_autoplaced yes)
 		(effects
@@
 		)
 		(property "Intersheetrefs" "${INTERSHEET_REFS}"
-			(at 183.8695 83.82 0)
+			(at 186.4095 83.82 0)
 			(effects
 				(font
@@
 	(global_label "DATA0"
 		(shape input)
-		(at 124.46 96.52 270)
+		(at 124.46 99.06 270)
 		(fields_autoplaced yes)
 		(effects
@@
 		)
 		(property "Intersheetrefs" "${INTERSHEET_REFS}"
-			(at 124.46 105.1295 90)
+			(at 124.46 107.6695 90)
 			(effects
 				(font
@@
 	(symbol
 		(lib_id "PCM_SparkFun-Capacitor:C")
-		(at 160.02 106.68 0)
+		(at 160.02 109.22 0)
 		(unit 1)
 		(exclude_from_sim no)
@@
 		(dnp no)
 		(property "Reference" "C18"
-			(at 162.814 105.664 0)
+			(at 162.814 108.204 0)
 			(effects
 				(font
@@
 		)
 		(property "Value" "2u2"
-			(at 162.814 107.696 0)
+			(at 162.814 110.236 0)
 			(effects
 				(font
@@
 		)
 		(property "Footprint" "Capacitor_SMD:C_0603_1608Metric"
-			(at 160.9852 118.11 0)
+			(at 160.9852 120.65 0)
 			(effects
 				(font
@@
 		)
 		(property "Datasheet" ""
-			(at 161.29 123.19 0)
+			(at 161.29 125.73 0)
 			(effects
 				(font
@@
 		)
 		(property "Description" "Unpolarized capacitor"
-			(at 160.02 125.73 0)
+			(at 160.02 128.27 0)
 			(effects
 				(font
@@
 	(symbol
 		(lib_id "power:GND")
-		(at 160.02 109.22 0)
+		(at 160.02 111.76 0)
 		(unit 1)
 		(exclude_from_sim no)
@@
 		(dnp no)
 		(property "Reference" "#PWR040"
-			(at 160.02 115.57 0)
+			(at 160.02 118.11 0)
 			(effects
 				(font
@@
 		)
 		(property "Value" "GND"
-			(at 160.02 113.03 0)
+			(at 160.02 115.57 0)
 			(effects
 				(font
@@
 		)
 		(property "Footprint" ""
-			(at 160.02 109.22 0)
+			(at 160.02 111.76 0)
 			(effects
 				(font
@@
 		)
 		(property "Datasheet" ""
-			(at 160.02 109.22 0)
+			(at 160.02 111.76 0)
 			(effects
 				(font
@@
 		)
 		(property "Description" "Power symbol creates a global label with name \"GND\" , ground"
-			(at 160.02 109.22 0)
+			(at 160.02 111.76 0)
 			(effects
 				(font
