File: KiCAD/sr42-udk-hotswap/sr42-udk-hotswap-argb.kicad_sch (KiCad schematic)
At the start: 92 parts, among them SW43 TPS22919

Commit message: wip-2025-11-24
Parts:
- removed SW43: TPS22919, Package_TO_SOT_SMD:SOT-363_SC-70-6, symbol ts-kicad-lib:TPS22919
- added SW44: TPS22810, Package_TO_SOT_SMD:SOT-23-6, symbol ts-kicad-lib:TPS22810
Connections:
- net +5V: no longer C45.2
- net GND: now also W27.3 (Vss), SW44.2 (GND); no longer W27.2 (Out)
- net LED_EN: now also SW44.3 (EN/VLO)
- net VLED: now also W27.1 (Vdd), SW44.6 (VOUT); no longer W27.4 (In)
- net at W28.4 (In): now also W27.2 (Out); no longer W27.1 (Vdd)
- net at W26.2 (Out): now also W27.4 (In); no longer W27.3 (Vss)
- net at R49.1: now also SW44.5 (QOD)
- new net +5V(b): C45.2, SW44.1 (VIN)
- no-connect marks 0 -> 1
Other:
- moved on the sheet: W27
Changed lines of the file:
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@@
 	(text "Power switch for\nper-key LEDs (3-44)"
 		(exclude_from_sim no)
-		(at 160.02 172.72 0)
+		(at 157.226 171.196 0)
 		(effects
 			(font
@@
 		(color 0 0 0 0)
 	)
+	(no_connect
+		(at 149.86 182.88)
+	)
 	(wire
 		(pts
@@
 	(wire
 		(pts
-			(xy 132.08 177.8) (xy 132.08 180.34)
-		)
-		(stroke
-			(width 0)
-			(type default)
-		)
-	)
-	(wire
-		(pts
 			(xy 86.36 129.54) (xy 93.98 129.54)
 		)
@@
 		)
 	)
+	(global_label "+5V(b)"
+		(shape input)
+		(at 132.08 180.34 180)
+		(fields_autoplaced yes)
+		(effects
+			(font
+				(size 1.27 1.27)
+			)
+			(justify right)
+		)
+		(property "Intersheetrefs" "${INTERSHEET_REFS}"
+			(at 122.3819 180.34 0)
+			(effects
+				(font
+					(size 1.27 1.27)
+				)
+				(justify right)
+				(hide yes)
+			)
+		)
+	)
 	(global_label "VLED"
 		(shape input)
@@
 		)
 	)
+	(global_label "+5V(b)"
+		(shape input)
+		(at 170.18 180.34 90)
+		(fields_autoplaced yes)
+		(effects
+			(font
+				(size 1.016 1.016)
+			)
+			(justify left)
+		)
+		(property "Intersheetrefs" "${INTERSHEET_REFS}"
+			(at 170.18 172.5819 90)
+			(effects
+				(font
+					(size 1.27 1.27)
+				)
+				(justify left)
+				(hide yes)
+			)
+		)
+	)
 	(global_label "VLED"
 		(shape input)
@@
 	(symbol
 		(lib_id "ts-keyboard-lib:SK6812MINI-E")
-		(at 119.38 81.28 270)
+		(at 119.38 81.28 0)
 		(unit 1)
 		(exclude_from_sim no)
@@
 		(fields_autoplaced yes)
 		(property "Reference" "W27"
-			(at 127 74.8598 90)
+			(at 127 74.8598 0)
 			(effects
 				(font
@@
 		)
 		(property "Value" "~"
-			(at 127 77.3998 90)
+			(at 127 77.3998 0)
 			(effects
 				(font
@@
 		)
 		(property "Footprint" "ts-keyboard-lib:SK6812MINI-E"
-			(at 112.776 81.28 0)
+			(at 119.38 87.884 0)
 			(effects
 				(font
@@
 		)
 		(property "Datasheet" "https://github.com/Tecsmith/ts-kicad-lib/blob/main/docs/sk6812mini-e-C5149201.pdf"
-			(at 110.744 81.28 0)
+			(at 119.38 89.916 0)
 			(effects
 				(font
@@
 	)
 	(symbol
-		(lib_id "ts-kicad-lib:TPS22919")
-		(at 142.24 182.88 0)
-		(unit 1)
-		(exclude_from_sim no)
-		(in_bom yes)
-		(on_board yes)
-		(dnp no)
-		(fields_autoplaced yes)
-		(property "Reference" "SW43"
-			(at 142.24 173.99 0)
-			(effects
-				(font
-					(size 1.27 1.27)
-				)
-			)
-		)
-		(property "Value" "TPS22919"
-			(at 142.24 176.53 0)
-			(effects
-				(font
-					(size 1.27 1.27)
-				)
-			)
-		)
-		(property "Footprint" "Package_TO_SOT_SMD:SOT-363_SC-70-6"
-			(at 142.24 194.31 0)
-			(effects
-				(font
-					(size 1.27 1.27)
-				)
-				(hide yes)
-			)
-		)
-		(property "Datasheet" "https://ti.com/lit/ds/symlink/tps22919.pdf"
-			(at 142.24 196.85 0)
-			(effects
-				(font
-					(size 1.27 1.27)
-				)
-				(hide yes)
-			)
-		)
-		(property "Description" "TPS22919 5.5 V, 1.5 A, 90-mΩ Self-Protected Load Switch with Controlled Rise Time"
-			(at 142.24 191.77 0)
-			(effects
-				(font
-					(size 1.27 1.27)
-				)
-				(hide yes)
-			)
-		)
-		(property "LCSC" "C2871558"
-			(at 142.24 199.39 0)
-			(effects
-				(font
-					(size 1.27 1.27)
-				)
-				(hide yes)
-			)
-		)
-		(pin "1"
-		)
-		(pin "3"
-		)
-		(pin "2"
-		)
-		(pin "6"
-		)
-		(pin "4"
-		)
-		(pin "5"
-		)
-		(instances
-			(project ""
-				(path "/f46a5539-adf6-4398-ac89-026a5789886b/927beec8-2af1-485b-83ac-8d4b31fb2213"
-					(reference "SW43")
-					(unit 1)
-				)
-			)
-		)
-	)
-	(symbol
 		(lib_id "power:GND")
 		(at 58.42 53.34 180)
@@
 	)
 	(symbol
-		(lib_id "power:+5V")
-		(at 132.08 177.8 0)
-		(unit 1)
-		(exclude_from_sim no)
-		(in_bom yes)
-		(on_board yes)
-		(dnp no)
-		(property "Reference" "#PWR067"
-			(at 132.08 181.61 0)
-			(effects
-				(font
-					(size 1.27 1.27)
-				)
-				(hide yes)
-			)
-		)
-		(property "Value" "+5V"
-			(at 132.08 174.244 0)
-			(effects
-				(font
-					(size 1.27 1.27)
-				)
-			)
-		)
-		(property "Footprint" ""
-			(at 132.08 177.8 0)
-			(effects
-				(font
-					(size 1.27 1.27)
-				)
-				(hide yes)
-			)
-		)
-		(property "Datasheet" ""
-			(at 132.08 177.8 0)
-			(effects
-				(font
-					(size 1.27 1.27)
-				)
-				(hide yes)
-			)
-		)
-		(property "Description" "Power symbol creates a global label with name \"+5V\""
-			(at 132.08 177.8 0)
-			(effects
-				(font
-					(size 1.27 1.27)
-				)
-				(hide yes)
-			)
-		)
-		(pin "1"
-		)
-		(instances
-			(project "sr42-udk-hotswap"
-				(path "/f46a5539-adf6-4398-ac89-026a5789886b/927beec8-2af1-485b-83ac-8d4b31fb2213"
-					(reference "#PWR067")
-					(unit 1)
-				)
-			)
-		)
-	)
-	(symbol
 		(lib_id "power:GND")
 		(at 99.06 86.36 0)
@@
 	)
 	(symbol
-		(lib_id "power:+5V")
-		(at 170.18 180.34 0)
-		(unit 1)
-		(exclude_from_sim no)
-		(in_bom yes)
-		(on_board yes)
-		(dnp no)
-		(property "Reference" "#PWR068"
-			(at 170.18 184.15 0)
-			(effects
-				(font
-					(size 1.27 1.27)
-				)
-				(hide yes)
-			)
-		)
-		(property "Value" "+5V"
-			(at 170.18 176.784 0)
-			(effects
-				(font
-					(size 1.27 1.27)
-				)
-			)
-		)
-		(property "Footprint" ""
-			(at 170.18 180.34 0)
-			(effects
-				(font
-					(size 1.27 1.27)
-				)
-				(hide yes)
-			)
-		)
-		(property "Datasheet" ""
-			(at 170.18 180.34 0)
-			(effects
-				(font
-					(size 1.27 1.27)
-				)
-				(hide yes)
-			)
-		)
-		(property "Description" "Power symbol creates a global label with name \"+5V\""
-			(at 170.18 180.34 0)
-			(effects
-				(font
-					(size 1.27 1.27)
-				)
-				(hide yes)
-			)
-		)
-		(pin "1"
-		)
-		(instances
-			(project "sr42-udk-hotswap"
-				(path "/f46a5539-adf6-4398-ac89-026a5789886b/927beec8-2af1-485b-83ac-8d4b31fb2213"
-					(reference "#PWR068")
-					(unit 1)
-				)
-			)
-		)
-	)
-	(symbol
 		(lib_id "power:GND")
 		(at 180.34 53.34 180)
@@
 					(unit 1)
 				)
+			)
+		)
+	)
+	(symbol
+		(lib_id "ts-kicad-lib:TPS22810")
+		(at 142.24 182.88 0)
+		(unit 1)
+		(exclude_from_sim no)
+		(in_bom yes)
+		(on_board yes)
+		(dnp no)
+		(fields_autoplaced yes)
+		(property "Reference" "SW44"
+			(at 142.24 173.99 0)
+			(effects
+				(font
+					(size 1.27 1.27)
+				)
+			)
+		)
+		(property "Value" "TPS22810"
+			(at 142.24 176.53 0)
+			(effects
+				(font
+					(size 1.27 1.27)
+				)
+			)
+		)
+		(property "Footprint" "Package_TO_SOT_SMD:SOT-23-6"
+			(at 142.24 194.31 0)
+			(effects
+				(font
+					(size 1.27 1.27)
+				)
+				(hide yes)
+			)
+		)
+		(property "Datasheet" "https://ti.com/lit/ds/symlink/tps22810.pdf"
+			(at 142.24 196.85 0)
+			(effects
+				(font
+					(size 1.27 1.27)
+				)
+				(hide yes)
+			)
+		)
+		(property "Description" "TPS22810, 2.7-18-V, 79-mΩ On-Resistance Load Switch With Thermal Protection"
+			(at 142.24 191.77 0)
+			(effects
+				(font
+					(size 1.27 1.27)
+				)
+				(hide yes)
+			)
+		)
+		(property "LCSC" "C205990"
+			(at 142.24 199.39 0)
+			(effects
+				(font
+					(size 1.27 1.27)
+				)
+				(hide yes)
+			)
+		)
+		(pin "3"
+		)
+		(pin "2"
+		)
+		(pin "6"
+		)
+		(pin "4"
+		)
+		(pin "5"
+		)
+		(pin "1"
+		)
+		(instances
+			(project ""
+				(path "/f46a5539-adf6-4398-ac89-026a5789886b/927beec8-2af1-485b-83ac-8d4b31fb2213"
+					(reference "SW44")
+					(unit 1)
+				)

Commit message: wip-2025-11-25
Parts:
- R49: footprint (none) -> Resistor_SMD:R_0603_1608Metric
- renumbered SW44 to RLY1
Changed lines of the file:
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@@
 			)
 		)
-		(property "Footprint" ""
+		(property "Footprint" "Resistor_SMD:R_0603_1608Metric"
 			(at 154.94 185.42 0)
 			(effects
@@
 		(dnp no)
 		(fields_autoplaced yes)
-		(property "Reference" "SW44"
+		(property "Reference" "RLY1"
 			(at 142.24 173.99 0)
 			(effects
@@
 			(project ""
 				(path "/f46a5539-adf6-4398-ac89-026a5789886b/927beec8-2af1-485b-83ac-8d4b31fb2213"
-					(reference "SW44")
+					(reference "RLY1")
 					(unit 1)
 				)

Commit message: june 2026 update
Parts:
- J1, W1, W10, W11, W12, W13, W14, W15, W16, W17, W18, W19, W2, W20, W21, W22, W23, W24, W25, W26, W27, W28, W29, W3, W30, W31, W32, W33, W34, W35, W36, W37, W38, W39, W4, W40, W41, W42, W43, W44, W5, W6, W7, W8, W9: value ~ -> (none)
