File: KiCAD/sr42-udk-hotswap/sr42-udk-hotswap-matrix.kicad_sch (KiCad schematic)
At the start: 44 parts

Commit message: wip-2025-11-24
Parts:
- added C52: 0-50u, Capacitor_SMD:C_0603_1608Metric, symbol ts-kicad-lib:C
- added C53: 100n, Capacitor_SMD:C_0603_1608Metric, symbol ts-kicad-lib:C
- added J7: ~, Connector_JST:JST_SH_SM02B-SRSS-TB_1x02-1MP_P1.00mm_Horizontal, symbol ts-kicad-lib:CONN_02
- added SW71: SW_DIP_x04, ts-kicad-lib:SW_DIP_SPSTx04, symbol Switch:SW_DIP_x04
- added U7: TTP223, Package_TO_SOT_SMD:SOT-23-6_Handsoldering, symbol ts-kicad-lib:TTP223
Connections:
- net +3.3V: now also C53.1, SW71.5, SW71.6, SW71.7, SW71.8, U7.5 (VDD)
- new net: J7.1, U7.3 (I)
- new net: C52.2, J7.2
- new net GND: C52.1, C53.2, U7.2 (VSS), U7.4 (AHLB), U7.6 (TOG)
- new net KD36: SW71.1
- new net KD37: SW71.2
- new net KD46: SW71.3
- new net KD47: SW71.4
- new net KT27: U7.1 (Q)
- no-connect marks 0 -> 1

Commit message: wip-2025-11-25
Parts:
- added J4: ~, Connector_PinHeader_2.54mm:PinHeader_1x02_P2.54mm_Vertical, symbol ts-kicad-lib:CONN_02
Connections:
- net +3.3V: now also J4.2
- new net KX57: J4.1
- no-connect marks 1 -> 2
Changed lines of the file:
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@@
 	)
 	(no_connect
+		(at 195.58 109.22)
+	)
+	(no_connect
 		(at 210.82 132.08)
 	)
@@
 		)
 	)
+	(global_label "KX57"
+		(shape input)
+		(at 193.04 106.68 180)
+		(fields_autoplaced yes)
+		(effects
+			(font
+				(size 1.27 1.27)
+			)
+			(justify right)
+		)
+		(property "Intersheetrefs" "${INTERSHEET_REFS}"
+			(at 185.1563 106.68 0)
+			(effects
+				(font
+					(size 1.27 1.27)
+				)
+				(justify right)
+				(hide yes)
+			)
+		)
+	)
 	(global_label "KD36"
 		(shape input)
@@
 	)
 	(symbol
+		(lib_id "power:+3.3V")
+		(at 193.04 104.14 90)
+		(unit 1)
+		(exclude_from_sim no)
+		(in_bom yes)
+		(on_board yes)
+		(dnp no)
+		(property "Reference" "#PWR067"
+			(at 196.85 104.14 0)
+			(effects
+				(font
+					(size 1.27 1.27)
+				)
+				(hide yes)
+			)
+		)
+		(property "Value" "+3.3V"
+			(at 189.738 102.108 90)
+			(effects
+				(font
+					(size 1.27 1.27)
+				)
+			)
+		)
+		(property "Footprint" ""
+			(at 193.04 104.14 0)
+			(effects
+				(font
+					(size 1.27 1.27)
+				)
+				(hide yes)
+			)
+		)
+		(property "Datasheet" ""
+			(at 193.04 104.14 0)
+			(effects
+				(font
+					(size 1.27 1.27)
+				)
+				(hide yes)
+			)
+		)
+		(property "Description" "Power symbol creates a global label with name \"+3.3V\""
+			(at 193.04 104.14 0)
+			(effects
+				(font
+					(size 1.27 1.27)
+				)
+				(hide yes)
+			)
+		)
+		(pin "1"
+		)
+		(instances
+			(project "sr42-udk-hotswap"
+				(path "/f46a5539-adf6-4398-ac89-026a5789886b/ae5e24a8-a0c4-4701-9208-d5e4602a2b27"
+					(reference "#PWR067")
+					(unit 1)
+				)
+			)
+		)
+	)
+	(symbol
 		(lib_id "ts-keyboard-lib:Momentary_Switch")
 		(at 58.42 53.34 0)
@@
 					(unit 1)
 				)
+			)
+		)
+	)
+	(symbol
+		(lib_id "ts-kicad-lib:CONN_02")
+		(at 195.58 106.68 0)
+		(unit 1)
+		(exclude_from_sim no)
+		(in_bom yes)
+		(on_board yes)
+		(dnp no)
+		(fields_autoplaced yes)
+		(property "Reference" "J4"
+			(at 199.39 104.4955 0)
+			(effects
+				(font
+					(size 1.27 1.27)
+				)
+				(justify left)
+			)
+		)
+		(property "Value" "~"
+			(at 199.39 107.0355 0)
+			(effects
+				(font
+					(size 1.27 1.27)
+				)
+				(justify left)
+			)
+		)
+		(property "Footprint" "Connector_PinHeader_2.54mm:PinHeader_1x02_P2.54mm_Vertical"
+			(at 195.58 106.68 0)
+			(effects
+				(font
+					(size 1.27 1.27)
+				)
+				(hide yes)
+			)
+		)
+		(property "Datasheet" ""
+			(at 195.58 106.68 0)
+			(effects
+				(font
+					(size 1.27 1.27)
+				)
+				(hide yes)
+			)
+		)
+		(property "Description" ""
+			(at 195.58 106.68 0)
+			(effects
+				(font
+					(size 1.27 1.27)
+				)
+				(hide yes)
+			)
+		)
+		(pin "2"
+		)
+		(pin "1"
+		)
+		(pin "MP"
+		)
+		(instances
+			(project ""
+				(path "/f46a5539-adf6-4398-ac89-026a5789886b/ae5e24a8-a0c4-4701-9208-d5e4602a2b27"
+					(reference "J4")
+					(unit 1)
+				)

Commit message: june 2026 update
Parts:
- J4, J7, ST1, ST2, SW1, SW10, SW11, SW12, SW13, SW14, SW15, SW16, SW17, SW18, SW19, SW2, SW20, SW21, SW22, SW23, SW24, SW25, SW26, SW27, SW28, SW29, SW3, SW30, SW31, SW32, SW33, SW34, SW35, SW36, SW37, SW38, SW39, SW4, SW40, SW41, SW42, SW5, SW6, SW7, SW8, SW9: value ~ -> (none)
