File: KiCAD/sr42-udk-hotswap/sr42-udk-hotswap.kicad_sch (KiCad schematic)
At the start: 31 parts, among them J2 5V, J3 ARGB, J4 QWIIC, J5 CONN, J6 SPI, Q1 2N7002, U1 MC74HC589AD, U2 MC74HC589AD, U3 MC74HC589AD, U4 MC74HC589AD, U5 MC74HC589AD, U6 MC74HC589AD

Commit message: wip-2025-11-24
Parts:
- removed J4: QWIIC, Connector_JST:JST_SH_SM04B-SRSS-TB_1x04-1MP_P1.00mm_Horizontal, symbol ts-kicad-lib:QWIIC
Connections:
- net SS is gone; now on net MATRIX_CS: J6.6
- net +5V: no longer J2.2
- net at R9.2: now also U5.5 (F); no longer U5.6 (G)
- net LATCH: now reaches Q1.3 (D), R13.1, U1.12 (LATCH), U1.13 (SS/~{PL}), U2.12 (LATCH), U2.13 (SS/~{PL}), U3.12 (LATCH), U3.13 (SS/~{PL}), U4.12 (LATCH), U4.13 (SS/~{PL}), U5.12 (LATCH), U5.13 (SS/~{PL}), U6.12 (LATCH), U6.13 (SS/~{PL})
- net at R9.1: now also U5.4 (E); no longer U5.7 (H)
- net at U5.1 (B): now also R10.1; no longer R10.3
- net at U5.3 (D): now also R10.3; no longer R10.1
- net at R9.4: now also U5.7 (H); no longer U5.4 (E)
- net at R9.3: now also U5.6 (G); no longer U5.5 (F)
- net CON1 renamed LED_EN
- net CON2: no longer names the net of J5.2
- net CON3: no longer names the net of J5.3
- net CON4: no longer names the net of J5.4
- net CON5: no longer names the net of J5.5
- net REG12 renamed SHFT-1-2
- net REG23 renamed SHFT-2-3
- net REG34 renamed SHFT-3-4
- net REG45 renamed SHFT-4-5
- net REG56 renamed SHFT-5-6
- new net +5V(b): J2.2
- no-connect marks 0 -> 4
Other:
- moved on the sheet: J2, J3, J5, J6

Commit message: wip-2025-11-25
Parts:
- added FID1, FID2, FID3: Fiducial, Fiducial:Fiducial_0.5mm_Mask1mm, symbol Mechanical:Fiducial
Connections:
- net MISO is gone; now on net PICO: U1.9 (QH)
- net K41: now also R10.1, U5.1 (B)
- net K42: now also R10.2, U5.2 (C)
- net K43: now also R10.3, U5.3 (D)
- net K44: now also R9.1, U5.4 (E)
- net K45: now also R9.2, U5.5 (F)
- net KD46: now also R9.3, U5.6 (G)
- net KD47: now also R9.4, U5.7 (H)
- net k40: now reaches R10.4, U5.15 (A)
- no-connect marks 4 -> 5

Commit message: wip-2025-11-27
Connections:
- net LED_EN: now also J5.3; no longer J5.1
Changed lines of the file:
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@@
 	)
 	(no_connect
-		(at 248.92 149.86)
+		(at 243.84 149.86)
 	)
 	(no_connect
@@
 	(global_label "LED_EN"
 		(shape input)
-		(at 243.84 149.86 90)
+		(at 248.92 149.86 90)
 		(fields_autoplaced yes)
 		(effects
@@
 		)
 		(property "Intersheetrefs" "${INTERSHEET_REFS}"
-			(at 243.84 139.9806 90)
+			(at 248.92 139.9806 90)
 			(effects
 				(font
