File: KiCAD/sr42-udk-hotswap-matrix.kicad_sch (KiCad schematic)
At the start: 50 parts, among them SW71 SW_DIP_x04, U7 TTP223

Commit message: updates
Connections:
- net GND: now also J7.MP
- net Touch: now reaches J7.1, U7.3 (I)
- no-connect marks 2 -> 1
Other:
- note added: "Optional DIP array"
- note added: "Optional Touch Sensor"
- moved on the sheet: C52, J7, SW71
