File: KiCAD/sr42-udk-hotswap.kicad_sch (KiCad schematic)
At the start: 33 parts, among them J2 5V, J3 ARGB, J5 CONN, J6 SPI, Q1 2N7002, U1 MC74HC589AD, U2 MC74HC589AD, U3 MC74HC589AD, U4 MC74HC589AD, U5 MC74HC589AD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

Commit message: updates
Parts:
- FID1, FID2, FID3: footprint Fiducial:Fiducial_0.5mm_Mask1mm -> ts-kicad-lib:Fiducial_0.5mm_Mask1mm_F
Other:
- moved on the sheet: FID1, FID2, FID3
Changed lines of the file:
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@@
 	(symbol
 		(lib_id "Mechanical:Fiducial")
-		(at 15.24 182.88 0)
+		(at 15.24 193.04 0)
 		(unit 1)
 		(body_style 1)
@@
 		(in_pos_files yes)
 		(dnp no)
-		(fields_autoplaced yes)
 		(property "Reference" "FID3"
-			(at 17.78 181.6099 0)
+			(at 17.78 193.04 0)
 			(show_name no)
 			(do_not_autoplace no)
@@
 		)
 		(property "Value" "Fiducial"
-			(at 17.78 184.1499 0)
+			(at 17.78 194.3099 0)
+			(hide yes)
 			(show_name no)
 			(do_not_autoplace no)
@@
 			)
 		)
-		(property "Footprint" "Fiducial:Fiducial_0.5mm_Mask1mm"
-			(at 15.24 182.88 0)
+		(property "Footprint" "ts-kicad-lib:Fiducial_0.5mm_Mask1mm_F"
+			(at 15.24 193.04 0)
 			(hide yes)
 			(show_name no)
@@
 		)
 		(property "Datasheet" ""
-			(at 15.24 182.88 0)
+			(at 15.24 193.04 0)
 			(hide yes)
 			(show_name no)
@@
 		)
 		(property "Description" "Fiducial Marker"
-			(at 15.24 182.88 0)
+			(at 15.24 193.04 0)
 			(hide yes)
 			(show_name no)
@@
 	(symbol
 		(lib_id "Mechanical:Fiducial")
-		(at 15.24 187.96 0)
+		(at 15.24 189.23 0)
 		(unit 1)
 		(body_style 1)
@@
 		(in_pos_files yes)
 		(dnp no)
-		(fields_autoplaced yes)
 		(property "Reference" "FID2"
-			(at 17.78 186.6899 0)
+			(at 17.78 189.23 0)
 			(show_name no)
 			(do_not_autoplace no)
@@
 		)
 		(property "Value" "Fiducial"
-			(at 17.78 189.2299 0)
+			(at 17.78 190.4999 0)
+			(hide yes)
 			(show_name no)
 			(do_not_autoplace no)
@@
 			)
 		)
-		(property "Footprint" "Fiducial:Fiducial_0.5mm_Mask1mm"
-			(at 15.24 187.96 0)
+		(property "Footprint" "ts-kicad-lib:Fiducial_0.5mm_Mask1mm_F"
+			(at 15.24 189.23 0)
 			(hide yes)
 			(show_name no)
@@
 		)
 		(property "Datasheet" ""
-			(at 15.24 187.96 0)
+			(at 15.24 189.23 0)
 			(hide yes)
 			(show_name no)
@@
 		)
 		(property "Description" "Fiducial Marker"
-			(at 15.24 187.96 0)
+			(at 15.24 189.23 0)
 			(hide yes)
 			(show_name no)
@@
 	(symbol
 		(lib_id "Mechanical:Fiducial")
-		(at 15.24 193.04 0)
+		(at 15.24 185.42 0)
 		(unit 1)
 		(body_style 1)
@@
 		(in_pos_files yes)
 		(dnp no)
-		(fields_autoplaced yes)
 		(property "Reference" "FID1"
-			(at 17.78 191.7699 0)
+			(at 17.78 185.42 0)
 			(show_name no)
 			(do_not_autoplace no)
@@
 		)
 		(property "Value" "Fiducial"
-			(at 17.78 194.3099 0)
+			(at 17.78 186.6899 0)
+			(hide yes)
 			(show_name no)
 			(do_not_autoplace no)
@@
 			)
 		)
-		(property "Footprint" "Fiducial:Fiducial_0.5mm_Mask1mm"
-			(at 15.24 193.04 0)
+		(property "Footprint" "ts-kicad-lib:Fiducial_0.5mm_Mask1mm_F"
+			(at 15.24 185.42 0)
 			(hide yes)
 			(show_name no)
@@
 		)
 		(property "Datasheet" ""
-			(at 15.24 193.04 0)
+			(at 15.24 185.42 0)
 			(hide yes)
 			(show_name no)
@@
 		)
 		(property "Description" "Fiducial Marker"
-			(at 15.24 193.04 0)
-			(hide yes)
-			(show_name no)
+			(at 15.24 185.42 0)
+			(hide yes)
+			(show_name no)
